File: camera.kicad_sch (KiCad schematic)
At the start: 1 part, among them J2 F32Q-1A7H1-11022

Commit message: restructured symbols, added footprints
Parts:
- J2: footprint (none) -> library:Hirose_FH12-22S-0.5SH_1x22-1MP_P0.50mm_Horizontal
Changed lines of the file:
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@@
 	)
 	(symbol
-		(lib_id "power:GND")
+		(lib_id "library:GND")
 		(at 153.67 125.73 0)
 		(unit 1)
@@
 			)
 		)
-		(property "Footprint" ""
+		(property "Footprint" "library:Hirose_FH12-22S-0.5SH_1x22-1MP_P0.50mm_Horizontal"
 			(at 166.37 97.79 0)
 			(effects
