File: CUTIE-CITRUS.kicad_pcb (KiCad board)
At the start: 2 copper layers, 48 parts, among them J1 F32Q-1A7H1-11022, J2 F32Q-1A7H1-11022, J3 Bus_M.2_Socket_M, J4 Hirose U.FL, U1 ASEK-32.768KHZ-L-R-T, U2 AP3441SHE-7B, U3 ICM-42688-P, U4 NEO-M8M

Commit message: prepared usb3, abstracted cameras, backplane connector
Parts:
- removed 3V3, 5V0, TP1, TP10, TP11, TP12, TP13, TP2, TP3, TP4, TP5, TP6, TP7, TP8, TP9: TestPoint, TestPoint:TestPoint_Pad_D1.0mm
- removed C1, C11, C9: 0.1uF, Capacitor_SMD:C_0402_1005Metric
- removed C10: 10nF, Capacitor_SMD:C_0402_1005Metric
- removed C12: 2.2uF, Capacitor_SMD:C_0402_1005Metric
- removed C2: 4.7nF, Capacitor_SMD:C_0402_1005Metric
- removed C3, C4, C5, C6, C7, C8: 10uF, Capacitor_SMD:C_0805_2012Metric
- removed CM5-1: 2x 10164227-1001A1RLF, library:RPi-CM5
- removed D1, D3: LED Green, LED_SMD:LED_0603_1608Metric
- removed D2: LED Red, LED_SMD:LED_0603_1608Metric
- removed D4: TPD1E05U06DPY, Package_SON:Texas_DPY0002A_0.6x1mm_P0.65mm
- removed J1, J2: F32Q-1A7H1-11022, library:Hirose_FH12-22S-0.5SH_1x22-1MP_P0.50mm_Horizontal
- removed J3: Bus_M.2_Socket_M, library:2230m2
- removed J4: Hirose U.FL, Connector_Coaxial:U.FL_Hirose_U.FL-R-SMT-1_Vertical
- removed R1, R4: 1k, Resistor_SMD:R_0402_1005Metric
- removed R2, R3, R7: 2.2K 1%, Resistor_SMD:R_0402_1005Metric
- removed R5: 100K 1%, Resistor_SMD:R_0402_1005Metric
- removed R6: 10K 1%, Resistor_SMD:R_0402_1005Metric
- removed R8: 1K, Resistor_SMD:R_0402_1005Metric
- removed U1: ASEK-32.768KHZ-L-R-T, Crystal:Crystal_SMD_3225-4Pin_3.2x2.5mm
- removed U2: AP3441SHE-7B, Package_DFN_QFN:DFN-8-1EP_2x2mm_P0.5mm_EP1.05x1.75mm
- removed U3: ICM-42688-P, Package_LGA:LGA-14_3x2.5mm_P0.5mm_LayoutBorder3x4y
- removed U4: NEO-M8M, RF_GPS:ublox_NEO

Commit message: un-abstraction, footprints, layout edge cuts
Parts:
- added 3V3: TestPoint, TestPoint:TestPoint_Pad_D2.0mm, F.Cu at (248.4, 124.5)
- added 3V3_M2: TestPoint, TestPoint:TestPoint_Pad_D1.0mm, F.Cu at (276.9, 82.3)
- added 5V0: TestPoint, TestPoint:TestPoint_Pad_D2.0mm, F.Cu at (248.4, 128.5)
- added C1: 10uF, Capacitor_SMD:C_0805_2012Metric, F.Cu at (273.5, 48.1)
- added C10: 0.1uF, Capacitor_SMD:C_0402_1005Metric, F.Cu at (264.0, 88.7)
- added C11: 2.2uF, Capacitor_SMD:C_0402_1005Metric, F.Cu at (264.0, 90.7)
- added C12: 10nF, Capacitor_SMD:C_0402_1005Metric, F.Cu at (264.0, 92.6)
- added C13: 47pF, Capacitor_SMD:C_0402_1005Metric, F.Cu at (264.0, 94.6)
- added C14: 0.1uF, Capacitor_SMD:C_0402_1005Metric, F.Cu at (264.0, 96.6)
- added C15: 2.2uF, Capacitor_SMD:C_0402_1005Metric, F.Cu at (264.0, 98.5)
- added C16: 1uF, Capacitor_SMD:C_0402_1005Metric, F.Cu at (264.0, 100.5)
- added C2: 10uF, Capacitor_SMD:C_0805_2012Metric, F.Cu at (273.5, 51.1)
- added C3: 0.1uF, Capacitor_SMD:C_0402_1005Metric, F.Cu at (275.6, 65.6)
- added C4: 0.1uF, Capacitor_SMD:C_0402_1005Metric, F.Cu at (275.6, 67.6)
- added C5: 4.7nF, Capacitor_SMD:C_0402_1005Metric, F.Cu at (275.6, 69.5)
- added C6: 10uF, Capacitor_SMD:C_0805_2012Metric, F.Cu at (273.5, 54.1)
- added C7: 10uF, Capacitor_SMD:C_0805_2012Metric, F.Cu at (273.5, 57.1)
- added C8: 10uF, Capacitor_SMD:C_0805_2012Metric, F.Cu at (273.5, 60.1)
- added C9: 10uF, Capacitor_SMD:C_0805_2012Metric, F.Cu at (273.5, 63.1)
- added CM5-1: 2x 10164227-1001A1RLF, library:RPi-CM5, F.Cu at (209.5, 70.5)
- added D1: LED Green, LED_SMD:LED_0603_1608Metric, F.Cu at (243.2, 69.9)
- added D2: LED Red, LED_SMD:LED_0603_1608Metric, F.Cu at (243.2, 72.5)
- added D3: LED Green, LED_SMD:LED_0603_1608Metric, F.Cu at (273.3, 82.1)
- added D4: TPD1E05U06DPY, Package_SON:Texas_DPY0002A_0.6x1mm_P0.65mm, F.Cu at (253.5, 106.2)
- added J1: F32Q-1A7H1-11022, library:Hirose_FH12-22S-0.5SH_1x22-1MP_P0.50mm_Horizontal, F.Cu at (201.8, 130.8)
- added J2: F32Q-1A7H1-11022, library:Hirose_FH12-22S-0.5SH_1x22-1MP_P0.50mm_Horizontal, F.Cu at (184.2, 130.8)
- added J3: Bus_M.2_Socket_M, library:2230m2, B.Cu at (193.0, 82.4)
- added J4: Hirose U.FL, Connector_Coaxial:U.FL_Hirose_U.FL-R-SMT-1_Vertical, F.Cu at (222.5, 122.0)
- added L1: 2.2uH, Capacitor_SMD:C_0402_1005Metric, F.Cu at (275.6, 71.5)
- added R1: 2.2K 1%, Resistor_SMD:R_0402_1005Metric, F.Cu at (242.6, 47.5)
- added R10: 2.2K 1%, Resistor_SMD:R_0402_1005Metric, F.Cu at (242.6, 57.5)
- added R11: 2.2K 1%, Resistor_SMD:R_0402_1005Metric, F.Cu at (242.6, 59.5)
- added R12: 2.2K 1%, Resistor_SMD:R_0402_1005Metric, F.Cu at (242.6, 61.5)
- added R2: 2.2K 1%, Resistor_SMD:R_0402_1005Metric, F.Cu at (242.6, 49.5)
- added R3: 1k, Resistor_SMD:R_0402_1005Metric, F.Cu at (242.6, 51.5)
- added R4: 1k, Resistor_SMD:R_0402_1005Metric, F.Cu at (242.6, 53.5)
- added R5: 100K 1%, Resistor_SMD:R_0402_1005Metric, F.Cu at (272.7, 65.6)
- added R6: 10K 1%, Resistor_SMD:R_0402_1005Metric, F.Cu at (272.7, 67.6)
- added R7: 2.2K 1%, Resistor_SMD:R_0402_1005Metric, F.Cu at (272.7, 69.6)
- added R8: 1K, Resistor_SMD:R_0402_1005Metric, F.Cu at (272.7, 71.6)
- added R9: 2.2K 1%, Resistor_SMD:R_0402_1005Metric, F.Cu at (242.6, 55.5)
- added TP1: TestPoint, TestPoint:TestPoint_Pad_D1.0mm, F.Cu at (247.9, 114.8)
- added TP10: TestPoint, TestPoint:TestPoint_Pad_D1.0mm, F.Cu at (257.1, 114.8)
- added TP11: TestPoint, TestPoint:TestPoint_Pad_D1.0mm, F.Cu at (257.1, 117.9)
- added TP12: TestPoint, TestPoint:TestPoint_Pad_D1.0mm, F.Cu at (257.1, 120.9)
- added TP13: TestPoint, TestPoint:TestPoint_Pad_D1.0mm, F.Cu at (260.1, 114.8)
- added TP14: TestPoint, TestPoint:TestPoint_Pad_D1.0mm, F.Cu at (260.1, 117.9)
- added TP15: TestPoint, TestPoint:TestPoint_Pad_D1.0mm, F.Cu at (260.1, 120.9)
- added TP16: TestPoint, TestPoint:TestPoint_Pad_D1.0mm, F.Cu at (242.7, 64.0)
- added TP17: TestPoint, TestPoint:TestPoint_Pad_D1.0mm, F.Cu at (242.7, 67.0)
- added TP18: TestPoint, TestPoint:TestPoint_Pad_D1.0mm, F.Cu at (266.9, 89.2)
- added TP19: TestPoint, TestPoint:TestPoint_Pad_D1.0mm, F.Cu at (266.9, 92.3)
- added TP2: TestPoint, TestPoint:TestPoint_Pad_D1.0mm, F.Cu at (247.9, 117.9)
- added TP20: TestPoint, TestPoint:TestPoint_Pad_D1.0mm, F.Cu at (266.9, 95.3)
- added TP3: TestPoint, TestPoint:TestPoint_Pad_D1.0mm, F.Cu at (247.9, 120.9)
- added TP4: TestPoint, TestPoint:TestPoint_Pad_D1.0mm, F.Cu at (251.0, 114.8)
- added TP5: TestPoint, TestPoint:TestPoint_Pad_D1.0mm, F.Cu at (251.0, 117.9)
- added TP6: TestPoint, TestPoint:TestPoint_Pad_D1.0mm, F.Cu at (251.0, 120.9)
- added TP7: TestPoint, TestPoint:TestPoint_Pad_D1.0mm, F.Cu at (254.1, 114.8)
- added TP8: TestPoint, TestPoint:TestPoint_Pad_D1.0mm, F.Cu at (254.1, 117.9)
- added TP9: TestPoint, TestPoint:TestPoint_Pad_D1.0mm, F.Cu at (254.1, 120.9)
- added U1: AP3441SHE-7B, Package_DFN_QFN:DFN-8-1EP_2x2mm_P0.5mm_EP1.05x1.75mm, F.Cu at (273.5, 79.1)
- added U2: ASEK-32.768KHZ-L-R-T, Crystal:Crystal_SMD_3225-4Pin_3.2x2.5mm, F.Cu at (273.9, 74.8)
- added U3: ICM-42688-P, Package_LGA:LGA-14_3x2.5mm_P0.5mm_LayoutBorder3x4y, F.Cu at (249.8, 107.3)
- added U4: NEO-M8M, RF_GPS:ublox_NEO, F.Cu at (224.5, 108.0)
Other:
- board outline added: 85 x 85 mm
