File: pcb/soc-flash.kicad_sch (KiCad schematic)
At the start: 4 parts, among them U3 S25FL128SAGNFV003

Commit message: added ddr3l
Parts:
- renumbered R5 to R6, R4 to R7, R1 to R8
Changed lines of the file:
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@@
 		(dnp no)
 		(fields_autoplaced yes)
-		(property "Reference" "R5"
+		(property "Reference" "R6"
 			(at 132.08 88.8999 0)
 			(effects
@@
 			(project "CUTIE-CITRUS"
 				(path "/875da261-7543-41df-9bd5-25bca104c872/ed92714e-f3d1-4199-bde0-4965b17657c9/dac30d8d-7a8b-44d0-9d3f-d7e0928892df"
-					(reference "R5")
+					(reference "R6")
 					(unit 1)
 				)
@@
 		(dnp no)
 		(fields_autoplaced yes)
-		(property "Reference" "#PWR04"
+		(property "Reference" "#PWR011"
 			(at 187.96 118.11 0)
 			(effects
@@
 			(project ""
 				(path "/875da261-7543-41df-9bd5-25bca104c872/ed92714e-f3d1-4199-bde0-4965b17657c9/dac30d8d-7a8b-44d0-9d3f-d7e0928892df"
-					(reference "#PWR04")
+					(reference "#PWR011")
 					(unit 1)
 				)
@@
 		(dnp no)
 		(fields_autoplaced yes)
-		(property "Reference" "R1"
+		(property "Reference" "R8"
 			(at 195.58 88.8999 0)
 			(effects
@@
 			(project "CUTIE-CITRUS"
 				(path "/875da261-7543-41df-9bd5-25bca104c872/ed92714e-f3d1-4199-bde0-4965b17657c9/dac30d8d-7a8b-44d0-9d3f-d7e0928892df"
-					(reference "R1")
+					(reference "R8")
 					(unit 1)
 				)
@@
 		(dnp no)
 		(fields_autoplaced yes)
-		(property "Reference" "R4"
+		(property "Reference" "R7"
 			(at 142.24 88.8999 0)
 			(effects
@@
 			(project "CUTIE-CITRUS"
 				(path "/875da261-7543-41df-9bd5-25bca104c872/ed92714e-f3d1-4199-bde0-4965b17657c9/dac30d8d-7a8b-44d0-9d3f-d7e0928892df"
-					(reference "R4")
+					(reference "R7")
 					(unit 1)
 				)
