File: pcb/soc-pwr.kicad_sch (KiCad schematic)
At the start: 1 part, among them U1 XC7Z020CLG484

Commit message: schematic structure, added qspi flash, pinout defs. mostly work on PS pinouts, defining comms. buses, still need to choose dram part, phys, camera/bus, power supply etc
Other:
- title: (none) -> CUTIE-CITRUS
Changed lines of the file:
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@@
 	(generator_version "9.0")
 	(paper "A4")
+	(title_block
+		(title "CUTIE-CITRUS")
+		(date "2026-01-21")
+		(rev "2.0")
+	)
 	(junction
 		(at 220.98 119.38)
