File: pcb/CUTIE-CITRUS.kicad_pcb (KiCad board)
At the start: 2 copper layers, 132 parts, among them J1 HIROSE_FH12-16S-0.5SH_55, U1 XC7Z020CLG484, U2 MT41K256M16, U3 S25FL128SAGNFV003, U5 RTL8211F-CG, U6 TCAN334

Commit message: power
Parts:
- added C1201: 39pF, Capacitor_SMD:C_0402_1005Metric, F.Cu at (99.6, 142.0)
- added C1202: 39pF, Capacitor_SMD:C_0402_1005Metric, F.Cu at (88.4, 142.0)
- added C1203: 0.1uF, Capacitor_SMD:C_0402_1005Metric, F.Cu at (90.2, 140.6)
- added C1204: 0.1uF, Capacitor_SMD:C_0402_1005Metric, F.Cu at (101.4, 140.6)
- added R1201: 37.4K, Resistor_SMD:R_0402_1005Metric, F.Cu at (87.4, 142.0)
- added R1202: 10K, Resistor_SMD:R_0402_1005Metric, F.Cu at (95.4, 137.8)
- added R1203: 20K, Resistor_SMD:R_0402_1005Metric, F.Cu at (98.6, 142.0)
- added R1204: 5.1K, Resistor_SMD:R_0402_1005Metric, F.Cu at (87.4, 140.0)
- added R1205: 10K, Resistor_SMD:R_0402_1005Metric, F.Cu at (84.2, 137.8)
- added R1206: 30K, Resistor_SMD:R_0402_1005Metric, F.Cu at (98.6, 140.0)
- added R1207: 0.003, Resistor_SMD:R_1206_3216Metric, F.Cu at (89.2, 144.2)
- added R1208: 10, Resistor_SMD:R_0402_1005Metric, F.Cu at (89.6, 142.0)
- added R1209: 10, Resistor_SMD:R_0402_1005Metric, F.Cu at (90.8, 142.0)
- added R1210: 10, Resistor_SMD:R_0402_1005Metric, F.Cu at (100.8, 142.0)
- added R1211: 0.01, Resistor_SMD:R_1206_3216Metric, F.Cu at (100.4, 144.2)
- added R1212: 10, Resistor_SMD:R_0402_1005Metric, F.Cu at (102.0, 142.0)
- added U1201: MPM3650, library:QFN-24_MPM3650_MNP, F.Cu at (84.2, 142.0)
- added U1202: MPM3650, library:QFN-24_MPM3650_MNP, F.Cu at (95.4, 142.0)
- R601, R602, R825: value 100 1% -> 100
- R826: value 240 1% -> 240
- moved R201 35.3 mm to (72.9, 153.8)
- moved R901 35.3 mm to (68.0, 153.8)
- moved R202 35.3 mm to (72.9, 155.8)
- moved R902 35.3 mm to (68.0, 155.8)
- moved R903 35.3 mm to (68.0, 157.8)
- moved C901 35.3 mm to (68.0, 159.8)
Connections:
- net /Debug Connectors/3V3_FD renamed /Debug Connectors/3V3_Z
- net /PHYs/3V3_FD renamed /PHYs/3V3_Z
- net /SoC/1V0_FD renamed /SoC/SoC Power/1V0_Z
- net /SoC/1V8_FD renamed /SoC/1V8_Z
- net /SoC/2V5_FD renamed /SoC/2V5_Z
- net /SoC/3V3_FD renamed /SoC/3V3_Z
- net /SoC/Flash Memory/3V3_FD renamed /SoC/Flash Memory/3V3_Z
