File: pcb/sch/backplane.kicad_sch (KiCad schematic)
At the start: 0 parts

Commit message: power
Changed lines of the file:
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@@
 		)
 	)
-	(hierarchical_label "12V0_RAW"
+	(hierarchical_label "VBUS"
 		(shape output)
 		(at 170.18 91.44 0)
