File: pcb/sch/main-pwr.kicad_sch (KiCad schematic)
At the start: 0 parts

Commit message: more pin definition pending define for how boot mode and power cycling will work, potential uc (stm32)
Changed lines of the file:
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@@
+	(wire
+		(pts
+			(xy 162.56 91.44) (xy 165.1 91.44)
+		)
+		(stroke
+			(width 0)
+			(type default)
+		)
+	)
 	(wire
 		(pts
@@
 		(effects
 			(font
+				(size 1.27 1.27)
+			)
+			(justify left)
+		)
+	)
+	(hierarchical_label "2V5_FD"
+		(shape output)
+		(at 165.1 91.44 0)
+		(effects
+			(font

Commit message: power
Parts:
- added C1201, C1202: 39pF, Capacitor_SMD:C_0402_1005Metric, symbol Device:C
- added C1203, C1204: 0.1uF, Capacitor_SMD:C_0402_1005Metric, symbol library:C
- added R1201: 37.4K, Resistor_SMD:R_0402_1005Metric, symbol Device:R_US
- added R1202, R1205: 10K, Resistor_SMD:R_0402_1005Metric, symbol Device:R_US
- added R1203: 20K, Resistor_SMD:R_0402_1005Metric, symbol Device:R_US
- added R1204: 5.1K, Resistor_SMD:R_0402_1005Metric, symbol Device:R_US
- added R1206: 30K, Resistor_SMD:R_0402_1005Metric, symbol Device:R_US
- added R1207: 0.003, Resistor_SMD:R_1206_3216Metric, symbol Device:R_US
- added R1208, R1209, R1210, R1212: 10, Resistor_SMD:R_0402_1005Metric, symbol library:R_US
- added R1211: 0.01, Resistor_SMD:R_1206_3216Metric, symbol Device:R_US
- added U1201, U1202: MPM3650, library:QFN-24_MPM3650_MNP, symbol library:MPM3650
Connections:
- new net: C1201.2, R1203.2, R1206.1, U1202.17 (FB)
- new net: C1202.2, R1201.2, R1204.1, U1201.17 (FB)
- new net: U1201.13 (SW), U1201.14 (SW), U1201.23 (SW), U1201.7 (SW), U1201.8 (SW)
- new net: U1202.13 (SW), U1202.14 (SW), U1202.23 (SW), U1202.7 (SW), U1202.8 (SW)
- new net 1V0: R1211.2, R1212.2
- new net 1V0_P: C1201.1, R1203.1, R1210.2, R1211.1, U1202.10 (OUT), U1202.11 (OUT), U1202.12 (OUT), U1202.9 (OUT)
- new net 1V0_PG: R1202.1, U1202.20 (PG), U1202.21 (PG)
- new net 1V0_SENS_N: C1204.2, R1212.1
- new net 1V0_SENS_P: C1204.1, R1210.1
- new net 5V0: R1207.2, R1209.2, U1202.22 (VIN)
- new net 5V0_P: C1202.1, R1201.1, R1207.1, R1208.2, U1201.10 (OUT), U1201.11 (OUT), U1201.12 (OUT), U1201.9 (OUT)
- new net 5V0_PG: R1205.1, U1201.20 (PG), U1201.21 (PG), U1202.16 (EN)
- new net 5V0_SENS_N: C1203.2, R1209.1
- new net 5V0_SENS_P: C1203.1, R1208.1
- new net GND: R1202.2, R1204.2, R1205.2, R1206.2, U1201.1 (PGND), U1201.18 (AGND), U1201.2 (PGND), U1201.24 (PGND), U1201.3 (PGND), U1201.4 (PGND), U1201.5 (PGND), U1201.6 (VCC), U1202.1 (PGND), U1202.18 (AGND), U1202.2 (PGND), U1202.24 (PGND), U1202.3 (PGND), U1202.4 (PGND), U1202.5 (PGND), U1202.6 (VCC)
- new net VBUS: U1201.16 (EN), U1201.22 (VIN)
Other:
- note added: "5A"
- note added: "6A"
- note added: "VBUS 5-12V NOMINAL?"
- note removed: "arbitrary abstraction"
- note removed: "maybe change 12v back to 5v depending on budget"
