File: pcb/sch/phy.kicad_sch (KiCad schematic)
At the start: 3 parts, among them U4 RTL8211F-CG, U5 TCAN334

Commit message: more pin definition pending define for how boot mode and power cycling will work, potential uc (stm32)
Parts:
- C1101: renamed from C6; Manufacturer KEMET -> (none); Manufacturer Product Number C0402C104K4RACTU -> (none); Part Description 0.1uF 10% 16V Ceramic Capacitor X7R 0402 (1005 Metric) -> (none)
- renumbered U4 to U5, U5 to U6
Changed lines of the file:
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@@
 		(dnp no)
 		(fields_autoplaced yes)
-		(property "Reference" "U5"
+		(property "Reference" "U6"
 			(at 215.9 96.52 0)
 			(show_name no)
@@
 		)
 		(instances
-			(project ""
+			(project "CUTIE-CITRUS"
 				(path "/875da261-7543-41df-9bd5-25bca104c872/35ff31e2-5977-44c6-8d54-93f4207ceb80"
-					(reference "U5")
+					(reference "U6")
 					(unit 1)
 				)
@@
 		(in_pos_files yes)
 		(dnp no)
-		(property "Reference" "C6"
+		(property "Reference" "C1101"
 			(at 196.85 121.92 0)
 			(show_name no)
@@
 			)
 		)
-		(property "Part Description" "	0.1uF 10% 16V Ceramic Capacitor X7R 0402 (1005 Metric)"
-			(at 200.66 123.19 0)
-			(hide yes)
-			(show_name no)
-			(do_not_autoplace no)
-			(effects
-				(font
-					(size 1.27 1.27)
-				)
-			)
-		)
-		(property "Manufacturer" "KEMET"
-			(at 200.66 123.19 0)
-			(hide yes)
-			(show_name no)
-			(do_not_autoplace no)
-			(effects
-				(font
-					(size 1.27 1.27)
-				)
-			)
-		)
-		(property "Manufacturer Product Number" "C0402C104K4RACTU"
+		(property "Part Description" ""
+			(at 200.66 123.19 0)
+			(hide yes)
+			(show_name no)
+			(do_not_autoplace no)
+			(effects
+				(font
+					(size 1.27 1.27)
+				)
+			)
+		)
+		(property "Manufacturer" ""
+			(at 200.66 123.19 0)
+			(hide yes)
+			(show_name no)
+			(do_not_autoplace no)
+			(effects
+				(font
+					(size 1.27 1.27)
+				)
+			)
+		)
+		(property "Manufacturer Product Number" ""
 			(at 200.66 123.19 0)
 			(hide yes)
@@
 			(project "CUTIE-CITRUS"
 				(path "/875da261-7543-41df-9bd5-25bca104c872/35ff31e2-5977-44c6-8d54-93f4207ceb80"
-					(reference "C6")
+					(reference "C1101")
 					(unit 1)
 				)
@@
 		(dnp no)
 		(fields_autoplaced yes)
-		(property "Reference" "#PWR013"
+		(property "Reference" "#PWR01103"
 			(at 231.14 135.89 0)
 			(hide yes)
@@
 			(project "CUTIE-CITRUS"
 				(path "/875da261-7543-41df-9bd5-25bca104c872/35ff31e2-5977-44c6-8d54-93f4207ceb80"
-					(reference "#PWR013")
+					(reference "#PWR01103")
 					(unit 1)
 				)
@@
 		(dnp no)
 		(fields_autoplaced yes)
-		(property "Reference" "#PWR014"
+		(property "Reference" "#PWR01101"
 			(at 71.12 146.05 0)
 			(hide yes)
@@
 		)
 		(instances
-			(project ""
+			(project "CUTIE-CITRUS"
 				(path "/875da261-7543-41df-9bd5-25bca104c872/35ff31e2-5977-44c6-8d54-93f4207ceb80"
-					(reference "#PWR014")
+					(reference "#PWR01101")
 					(unit 1)
 				)
@@
 		(dnp no)
 		(fields_autoplaced yes)
-		(property "Reference" "#PWR012"
+		(property "Reference" "#PWR01102"
 			(at 200.66 135.89 0)
 			(hide yes)
@@
 			(project "CUTIE-CITRUS"
 				(path "/875da261-7543-41df-9bd5-25bca104c872/35ff31e2-5977-44c6-8d54-93f4207ceb80"
-					(reference "#PWR012")
+					(reference "#PWR01102")
 					(unit 1)
 				)
@@
 		(dnp no)
 		(fields_autoplaced yes)
-		(property "Reference" "U4"
+		(property "Reference" "U5"
 			(at 93.98 55.88 0)
 			(show_name no)
@@
 		)
 		(instances
-			(project ""
+			(project "CUTIE-CITRUS"
 				(path "/875da261-7543-41df-9bd5-25bca104c872/35ff31e2-5977-44c6-8d54-93f4207ceb80"
-					(reference "U4")
+					(reference "U5")
 					(unit 1)
 				)

Commit message: power
Connections:
- net 3V3_FD renamed 3V3_Z
Changed lines of the file:
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@@
 		)
 	)
-	(hierarchical_label "3V3_FD"
+	(hierarchical_label "3V3_Z"
 		(shape input)
 		(at 187.96 116.84 180)
