File: pcb/sch/soc-1.kicad_sch (KiCad schematic)
At the start: 18 parts, among them U1 XC7Z020CLG484

Commit message: power
Connections:
- net 1V8_FD renamed 1V8_Z
- net 2V5_FD renamed 2V5_Z
- net 3V3_FD renamed 3V3_Z
Changed lines of the file:
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@@
 		)
 	)
-	(hierarchical_label "1V8_FD"
+	(hierarchical_label "1V8_Z"
 		(shape input)
 		(at 236.22 81.28 0)
@@
 		)
 	)
-	(hierarchical_label "3V3_FD"
+	(hierarchical_label "3V3_Z"
 		(shape input)
 		(at 264.16 25.4 0)
@@
 		)
 	)
-	(hierarchical_label "2V5_FD"
+	(hierarchical_label "2V5_Z"
 		(shape input)
 		(at 68.58 154.94 0)
@@
 		)
 	)
-	(hierarchical_label "2V5_FD"
-		(shape input)
-		(at 248.92 116.84 0)
-		(effects
-			(font
-				(size 1.27 1.27)
-			)
-			(justify left)
-		)
-	)
-	(hierarchical_label "3V3_FD"
+	(hierarchical_label "3V3_Z"
 		(shape input)
 		(at 248.92 139.7 0)
@@
 		)
 	)
-	(hierarchical_label "3V3_FD"
+	(hierarchical_label "3V3_Z"
 		(shape input)
 		(at 236.22 48.26 0)
@@
 		)
 	)
-	(hierarchical_label "3V3_FD"
+	(hierarchical_label "3V3_Z"
 		(shape input)
 		(at 162.56 154.94 0)
 		(effects
 			(font
+				(size 1.27 1.27)
+			)
+			(justify left)
+		)
+	)
+	(hierarchical_label "2V5_Z"
+		(shape input)
+		(at 248.92 116.84 0)
+		(effects
+			(font
