File: pcb/sch/soc-2.kicad_sch (KiCad schematic)
At the start: 1 part, among them U1 XC7Z020CLG484

Commit message: more pin definition pending define for how boot mode and power cycling will work, potential uc (stm32)
Parts:
- removed U1: XC7Z020CLG484, Package_BGA:Xilinx_CLG484_CLG485, symbol library:XC7Z020CLG484
- added C401, C402: 47uF, Capacitor_SMD:C_0805_2012Metric, symbol library:C
- added C403, C404, C405, C406: 4.7uF, Capacitor_SMD:C_0402_1005Metric, symbol library:C
- added C407, C408, C409, C410, C411, C412, C413, C414: 470nF, Capacitor_SMD:C_0402_1005Metric, symbol library:C
- added U1: XC7Z020CLG484, Package_BGA:Xilinx_CLG484_CLG485, symbol library:XC7Z020CLG484
Connections:
- new net: C402.2, C404.2, C406.2, C408.2, C410.2, C412.2, C414.2
- new net: C401.2, C403.2, C405.2, C407.2, C409.2, C411.2, C413.2
- new net GND: C401.1, C402.1, C403.1, C404.1, C405.1, C406.1, C407.1, C408.1, C409.1, C410.1, C411.1, C412.1, C413.1, C414.1
