File: pcb/sch/soc-ddr.kicad_sch (KiCad schematic)
At the start: 1 part, among them U1 XC7Z020CLG484

Commit message: more pin definition pending define for how boot mode and power cycling will work, potential uc (stm32)
Parts:
- removed U1: XC7Z020CLG484, Package_BGA:Xilinx_CLG484_CLG485, symbol library:XC7Z020CLG484
- added C601, C602, C603, C604: 470nF, Capacitor_SMD:C_0402_1005Metric, symbol library:C
- added C605: 4.7uF, Capacitor_SMD:C_0402_1005Metric, symbol library:C
- added C606: 100uF, Capacitor_SMD:C_1210_3225Metric, symbol library:C
- added C607, C608: 0.1uF, Capacitor_SMD:C_0402_1005Metric, symbol library:C
- added R601, R602: 100 1%, Resistor_SMD:R_0402_1005Metric, symbol Device:R_US
- added R603: 4.7K, Resistor_SMD:R_0402_1005Metric, symbol Device:R_US
- added U1: XC7Z020CLG484, Package_BGA:Xilinx_CLG484_CLG485, symbol library:XC7Z020CLG484
Connections:
- new net 0V675_REF: C607.2, C608.2, U1.H7 (PS_DDR_VREF0_502), U1.P7 (PS_DDR_VREF1_502)
- new net 1V35_DDR: C601.2, C602.2, C603.2, C604.2, C605.2, C606.2, R601.1, U1.E2 (VCCO_DDR_502), U1.F5 (VCCO_DDR_502), U1.H1 (VCCO_DDR_502), U1.J4 (VCCO_DDR_502), U1.K7 (VCCO_DDR_502), U1.M3 (VCCO_DDR_502), U1.N6 (VCCO_DDR_502), U1.R2 (VCCO_DDR_502), U1.V1 (VCCO_DDR_502)
- new net DDR_A0: U1.M4 (PS_DDR_A0_502)
- new net DDR_A1: U1.M5 (PS_DDR_A1_502)
- new net DDR_A10: U1.J3 (PS_DDR_A10_502)
- new net DDR_A11: U1.G5 (PS_DDR_A11_502)
- new net DDR_A12: U1.H4 (PS_DDR_A12_502)
- new net DDR_A13: U1.F4 (PS_DDR_A13_502)
- new net DDR_A14: U1.G4 (PS_DDR_A14_502)
- new net DDR_A2: U1.K4 (PS_DDR_A2_502)
- new net DDR_A3: U1.L4 (PS_DDR_A3_502)
- new net DDR_A4: U1.K6 (PS_DDR_A4_502)
- new net DDR_A5: U1.K5 (PS_DDR_A5_502)
- new net DDR_A6: U1.J7 (PS_DDR_A6_502)
- new net DDR_A7: U1.J6 (PS_DDR_A7_502)
- new net DDR_A8: U1.J5 (PS_DDR_A8_502)
- new net DDR_A9: U1.H5 (PS_DDR_A9_502)
- new net DDR_BA0: U1.L7 (PS_DDR_BA0_502)
- new net DDR_BA1: U1.L6 (PS_DDR_BA1_502)
- new net DDR_BA2: U1.M6 (PS_DDR_BA2_502)
- new net DDR_CAS: U1.P3 (PS_DDR_CAS_B_502)
- new net DDR_CKE: U1.V3 (PS_DDR_CKE_502)
- new net DDR_CK_N: U1.N5 (PS_DDR_CKN_502)
- new net DDR_CK_P: U1.N4 (PS_DDR_CKP_502)
- new net DDR_CS: U1.P6 (PS_DDR_CS_B_502)
- new net DDR_DM0: U1.B1 (PS_DDR_DM0_502)
- new net DDR_DM1: U1.H3 (PS_DDR_DM1_502)
- new net DDR_DM2: U1.P1 (PS_DDR_DM2_502)
- new net DDR_DM3: U1.AA2 (PS_DDR_DM3_502)
- new net DDR_DQ0: U1.D1 (PS_DDR_DQ0_502)
- new net DDR_DQ1: U1.C3 (PS_DDR_DQ1_502)
- new net DDR_DQ10: U1.L1 (PS_DDR_DQ10_502)
- new net DDR_DQ11: U1.L2 (PS_DDR_DQ11_502)
- new net DDR_DQ12: U1.L3 (PS_DDR_DQ12_502)
- new net DDR_DQ13: U1.K1 (PS_DDR_DQ13_502)
- new net DDR_DQ14: U1.J1 (PS_DDR_DQ14_502)
- new net DDR_DQ15: U1.K3 (PS_DDR_DQ15_502)
- new net DDR_DQ16: U1.M1 (PS_DDR_DQ16_502)
- new net DDR_DQ17: U1.T3 (PS_DDR_DQ17_502)
- new net DDR_DQ18: U1.N3 (PS_DDR_DQ18_502)
- new net DDR_DQ19: U1.T1 (PS_DDR_DQ19_502)
- new net DDR_DQ2: U1.B2 (PS_DDR_DQ2_502)
- new net DDR_DQ20: U1.R3 (PS_DDR_DQ20_502)
- new net DDR_DQ21: U1.T2 (PS_DDR_DQ21_502)
- new net DDR_DQ22: U1.M2 (PS_DDR_DQ22_502)
- new net DDR_DQ23: U1.R1 (PS_DDR_DQ23_502)
- new net DDR_DQ24: U1.AA3 (PS_DDR_DQ24_502)
- new net DDR_DQ25: U1.U1 (PS_DDR_DQ25_502)
- new net DDR_DQ26: U1.AA1 (PS_DDR_DQ26_502)
- new net DDR_DQ27: U1.U2 (PS_DDR_DQ27_502)
- new net DDR_DQ28: U1.W1 (PS_DDR_DQ28_502)
- new net DDR_DQ29: U1.Y3 (PS_DDR_DQ29_502)
- new net DDR_DQ3: U1.D3 (PS_DDR_DQ3_502)
- new net DDR_DQ30: U1.W3 (PS_DDR_DQ30_502)
- new net DDR_DQ31: U1.Y1 (PS_DDR_DQ31_502)
- new net DDR_DQ4: U1.E3 (PS_DDR_DQ4_502)
- new net DDR_DQ5: U1.E1 (PS_DDR_DQ5_502)
- new net DDR_DQ6: U1.F2 (PS_DDR_DQ6_502)
- new net DDR_DQ7: U1.F1 (PS_DDR_DQ7_502)
- new net DDR_DQ8: U1.G2 (PS_DDR_DQ8_502)
- new net DDR_DQ9: U1.G1 (PS_DDR_DQ9_502)
- new net DDR_DQS_0_N: U1.D2 (PS_DDR_DQS_N0_502)
- new net DDR_DQS_0_P: U1.C2 (PS_DDR_DQS_P0_502)
- new net DDR_DQS_1_N: U1.J2 (PS_DDR_DQS_N1_502)
- new net DDR_DQS_1_P: U1.H2 (PS_DDR_DQS_P1_502)
- new net DDR_DRST: R603.1, U1.F3 (PS_DDR_DRST_B_502)
- new net DDR_ODT: U1.P5 (PS_DDR_ODT_502)
- new net DDR_RAS: U1.R5 (PS_DDR_RAS_B_502)
- new net DDR_VRN: R602.1, U1.M7 (PS_DDR_VRN_502)
- new net DDR_VRP: R601.2, U1.N7 (PS_DDR_VRP_502)
- new net DDR_WE: U1.R4 (PS_DDR_WE_B_502)
- new net GND: C601.1, C602.1, C603.1, C604.1, C605.1, C606.1, C607.1, C608.1, R602.2, R603.2
Other:
- note added: "Byte 0"
- note added: "Byte 1"

Commit message: byte swapping and rough layout
Connections:
- net DDR_DM0: now also U1.H3 (PS_DDR_DM1_502); no longer U1.B1 (PS_DDR_DM0_502)
- net DDR_DM1: now also U1.B1 (PS_DDR_DM0_502); no longer U1.H3 (PS_DDR_DM1_502)
- net DDR_DQ0: now also U1.G2 (PS_DDR_DQ8_502); no longer U1.D1 (PS_DDR_DQ0_502)
- net DDR_DQ1: now also U1.G1 (PS_DDR_DQ9_502); no longer U1.C3 (PS_DDR_DQ1_502)
- net DDR_DQ10: now also U1.B2 (PS_DDR_DQ2_502); no longer U1.L1 (PS_DDR_DQ10_502)
- net DDR_DQ11: now also U1.D3 (PS_DDR_DQ3_502); no longer U1.L2 (PS_DDR_DQ11_502)
- net DDR_DQ12: now also U1.E3 (PS_DDR_DQ4_502); no longer U1.L3 (PS_DDR_DQ12_502)
- net DDR_DQ13: now also U1.E1 (PS_DDR_DQ5_502); no longer U1.K1 (PS_DDR_DQ13_502)
- net DDR_DQ14: now also U1.F2 (PS_DDR_DQ6_502); no longer U1.J1 (PS_DDR_DQ14_502)
- net DDR_DQ15: now also U1.F1 (PS_DDR_DQ7_502); no longer U1.K3 (PS_DDR_DQ15_502)
- net DDR_DQ2: now also U1.L1 (PS_DDR_DQ10_502); no longer U1.B2 (PS_DDR_DQ2_502)
- net DDR_DQ3: now also U1.L2 (PS_DDR_DQ11_502); no longer U1.D3 (PS_DDR_DQ3_502)
- net DDR_DQ4: now also U1.L3 (PS_DDR_DQ12_502); no longer U1.E3 (PS_DDR_DQ4_502)
- net DDR_DQ5: now also U1.K1 (PS_DDR_DQ13_502); no longer U1.E1 (PS_DDR_DQ5_502)
- net DDR_DQ6: now also U1.J1 (PS_DDR_DQ14_502); no longer U1.F2 (PS_DDR_DQ6_502)
- net DDR_DQ7: now also U1.K3 (PS_DDR_DQ15_502); no longer U1.F1 (PS_DDR_DQ7_502)
- net DDR_DQ8: now also U1.D1 (PS_DDR_DQ0_502); no longer U1.G2 (PS_DDR_DQ8_502)
- net DDR_DQ9: now also U1.C3 (PS_DDR_DQ1_502); no longer U1.G1 (PS_DDR_DQ9_502)
- net DDR_DQS_0_N: now also U1.J2 (PS_DDR_DQS_N1_502); no longer U1.D2 (PS_DDR_DQS_N0_502)
- net DDR_DQS_0_P: now also U1.H2 (PS_DDR_DQS_P1_502); no longer U1.C2 (PS_DDR_DQS_P0_502)
- net DDR_DQS_1_N: now also U1.D2 (PS_DDR_DQS_N0_502); no longer U1.J2 (PS_DDR_DQS_N1_502)
- net DDR_DQS_1_P: now also U1.C2 (PS_DDR_DQS_P0_502); no longer U1.H2 (PS_DDR_DQS_P1_502)
Changed lines of the file:
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@@
 	(text "Byte 1"
 		(exclude_from_sim no)
-		(at 208.28 63.5 0)
+		(at 205.74 40.64 0)
 		(effects
 			(font
@@
 	(text "Byte 0"
 		(exclude_from_sim no)
-		(at 208.28 40.64 0)
+		(at 205.74 63.5 0)
 		(effects
 			(font
@@
 	(polyline
 		(pts
-			(xy 205.74 30.48) (xy 205.74 50.8)
+			(xy 203.2 53.34) (xy 203.2 73.66)
 		)
 		(stroke
@@
 	(polyline
 		(pts
-			(xy 203.2 50.8) (xy 205.74 50.8)
+			(xy 200.66 73.66) (xy 203.2 73.66)
 		)
 		(stroke
@@
 	(polyline
 		(pts
-			(xy 203.2 53.34) (xy 205.74 53.34)
+			(xy 200.66 30.48) (xy 203.2 30.48)
 		)
 		(stroke
@@
 	(polyline
 		(pts
-			(xy 203.2 73.66) (xy 205.74 73.66)
+			(xy 200.66 50.8) (xy 203.2 50.8)
 		)
 		(stroke
@@
 	(polyline
 		(pts
-			(xy 203.2 30.48) (xy 205.74 30.48)
+			(xy 200.66 53.34) (xy 203.2 53.34)
 		)
 		(stroke
@@
 	(polyline
 		(pts
-			(xy 205.74 53.34) (xy 205.74 73.66)
+			(xy 203.2 30.48) (xy 203.2 50.8)
 		)
 		(stroke
@@
 		)
 	)
-	(label "DDR_DM1"
-		(at 81.28 116.84 0)
-		(effects
-			(font
-				(size 1.27 1.27)
-			)
-			(justify left bottom)
-		)
-	)
 	(label "DDR_A11"
 		(at 81.28 60.96 0)
@@
 		)
 	)
+	(label "DDR_DQ3"
+		(at 192.8733 63.5 180)
+		(effects
+			(font
+				(size 1.27 1.27)
+			)
+			(justify right bottom)
+		)
+	)
+	(label "DDR_DM1"
+		(at 81.28 106.68 0)
+		(effects
+			(font
+				(size 1.27 1.27)
+			)
+			(justify left bottom)
+		)
+	)
 	(label "DDR_DQ19"
 		(at 193.04 86.36 180)
@@
 		)
 	)
-	(label "DDR_DQ0"
-		(at 193.04 33.02 180)
-		(effects
-			(font
-				(size 1.27 1.27)
-			)
-			(justify right bottom)
-		)
-	)
 	(label "DDR_DQ16"
 		(at 193.04 78.74 180)
@@
 	)
 	(label "DDR_DQ1"
-		(at 193.04 35.56 180)
+		(at 192.8733 58.42 180)
 		(effects
 			(font
@@
 		)
 	)
+	(label "DDR_DQ0"
+		(at 192.8733 55.88 180)
+		(effects
+			(font
+				(size 1.27 1.27)
+			)
+			(justify right bottom)
+		)
+	)
 	(label "DDR_A9"
 		(at 81.28 55.88 0)
@@
 		)
 	)
+	(label "DDR_DQ11"
+		(at 193.04 40.64 180)
+		(effects
+			(font
+				(size 1.27 1.27)
+			)
+			(justify right bottom)
+		)
+	)
 	(label "DDR_DQ26"
 		(at 193.04 106.68 180)
@@
 		)
 	)
-	(label "DDR_DQ10"
-		(at 193.04 60.96 180)
-		(effects
-			(font
-				(size 1.27 1.27)
-			)
-			(justify right bottom)
+	(label "DDR_DQ15"
+		(at 193.04 50.8 180)
+		(effects
+			(font
+				(size 1.27 1.27)
+			)
+			(justify right bottom)
+		)
+	)
+	(label "DDR_DM0"
+		(at 81.1097 116.84 0)
+		(effects
+			(font
+				(size 1.27 1.27)
+			)
+			(justify left bottom)
 		)
 	)
@@
 		)
 	)
+	(label "DDR_DQ4"
+		(at 192.8733 66.04 180)
+		(effects
+			(font
+				(size 1.27 1.27)
+			)
+			(justify right bottom)
+		)
+	)
 	(label "DDR_A0"
 		(at 81.28 33.02 0)
@@
 		)
 	)
+	(label "DDR_DQ14"
+		(at 193.04 48.26 180)
+		(effects
+			(font
+				(size 1.27 1.27)
+			)
+			(justify right bottom)
+		)
+	)
+	(label "DDR_DQ2"
+		(at 192.8733 60.96 180)
+		(effects
+			(font
+				(size 1.27 1.27)
+			)
+			(justify right bottom)
+		)
+	)
 	(label "DDR_DQ21"
 		(at 193.04 91.44 180)
@@
 		)
 	)
+	(label "DDR_DQ6"
+		(at 192.8733 71.12 180)
+		(effects
+			(font
+				(size 1.27 1.27)
+			)
+			(justify right bottom)
+		)
+	)
 	(label "DDR_DQ23"
 		(at 193.04 96.52 180)
@@
 		)
 	)
-	(label "DDR_DQ7"
-		(at 193.04 50.8 180)
-		(effects
-			(font
-				(size 1.27 1.27)
-			)
-			(justify right bottom)
-		)
-	)
-	(label "DDR_DQ5"
-		(at 193.04 45.72 180)
+	(label "DDR_DQ10"
+		(at 193.04 38.1 180)
 		(effects
 			(font
@@
 		)
 	)
-	(label "DDR_DQ14"
-		(at 193.04 71.12 180)
-		(effects
-			(font
-				(size 1.27 1.27)
-			)
-			(justify right bottom)
-		)
-	)
-	(label "DDR_DQ15"
-		(at 193.04 73.66 180)
+	(label "DDR_DQ8"
+		(at 193.04 33.02 180)
+		(effects
+			(font
+				(size 1.27 1.27)
+			)
+			(justify right bottom)
+		)
+	)
+	(label "DDR_DQ9"
+		(at 193.04 35.56 180)
 		(effects
 			(font
@@
 		)
 	)
-	(label "DDR_DQ13"
-		(at 193.04 68.58 180)
-		(effects
-			(font
-				(size 1.27 1.27)
-			)
-			(justify right bottom)
-		)
-	)
 	(label "DDR_BA0"
 		(at 81.28 73.66 0)
@@
 		)
 	)
-	(label "DDR_DQ8"
-		(at 193.04 55.88 180)
-		(effects
-			(font
-				(size 1.27 1.27)
-			)
-			(justify right bottom)
-		)
-	)
 	(label "DDR_DQ29"
 		(at 193.04 114.3 180)
@@
 		)
 	)
+	(label "DDR_DQ5"
+		(at 192.8733 68.58 180)
+		(effects
+			(font
+				(size 1.27 1.27)
+			)
+			(justify right bottom)
+		)
+	)
 	(label "DDR_BA1"
 		(at 81.28 76.2 0)
@@
 		)
 	)
+	(label "DDR_DQ7"
+		(at 192.8733 73.66 180)
+		(effects
+			(font
+				(size 1.27 1.27)
+			)
+			(justify right bottom)
+		)
+	)
+	(label "DDR_DQ12"
+		(at 193.04 43.18 180)
+		(effects
+			(font
+				(size 1.27 1.27)
+			)
+			(justify right bottom)
+		)
+	)
 	(label "DDR_DQ31"
 		(at 193.04 119.38 180)
@@
 		)
 	)
-	(label "DDR_DQ6"
-		(at 193.04 48.26 180)
-		(effects
-			(font
-				(size 1.27 1.27)
-			)
-			(justify right bottom)
-		)
-	)
 	(label "DDR_A13"
 		(at 81.28 66.04 0)
@@
 		)
 	)
-	(label "DDR_DQ3"
-		(at 193.04 40.64 180)
-		(effects
-			(font
-				(size 1.27 1.27)
-			)
-			(justify right bottom)
-		)
-	)
 	(label "DDR_DQ18"
 		(at 193.04 83.82 180)
@@
 		)
 	)
-	(label "DDR_DQ11"
-		(at 193.04 63.5 180)
-		(effects
-			(font
-				(size 1.27 1.27)
-			)
-			(justify right bottom)
-		)
-	)
-	(label "DDR_DQ2"
-		(at 193.04 38.1 180)
-		(effects
-			(font
-				(size 1.27 1.27)
-			)
-			(justify right bottom)
-		)
-	)
-	(label "DDR_DQ9"
-		(at 193.04 58.42 180)
-		(effects
-			(font
-				(size 1.27 1.27)
-			)
-			(justify right bottom)
-		)
-	)
-	(label "DDR_DQ12"
-		(at 193.04 66.04 180)
+	(label "DDR_DQ13"
+		(at 193.04 45.72 180)
 		(effects
 			(font
@@
 	(label "DDR_A12"
 		(at 81.28 63.5 0)
-		(effects
-			(font
-				(size 1.27 1.27)
-			)
-			(justify left bottom)
-		)
-	)
-	(label "DDR_DQ4"
-		(at 193.04 43.18 180)
-		(effects
-			(font
-				(size 1.27 1.27)
-			)
-			(justify right bottom)
-		)
-	)
-	(label "DDR_DM0"
-		(at 81.28 106.68 0)
 		(effects
 			(font
@@
 		)
 	)
-	(hierarchical_label "DDR_DQS_1_P"
-		(shape bidirectional)
-		(at 101.6 119.38 180)
-		(effects
-			(font
-				(size 1.27 1.27)
-			)
-			(justify right)
-		)
-	)
 	(hierarchical_label "DDR_RAS"
 		(shape input)
@@
 	(hierarchical_label "DDR_DQS_1_N"
 		(shape bidirectional)
-		(at 101.6 121.92 180)
+		(at 101.6 111.76 180)
 		(effects
 			(font
@@
 		)
 	)
+	(hierarchical_label "DDR_DQS_0_P"
+		(shape bidirectional)
+		(at 101.6 119.38 180)
+		(effects
+			(font
+				(size 1.27 1.27)
+			)
+			(justify right)
+		)
+	)
 	(hierarchical_label "DDR_DM[0..3]"
 		(shape output)
@@
 	(hierarchical_label "DDR_DQS_0_N"
 		(shape bidirectional)
-		(at 101.6 111.76 180)
+		(at 101.6 121.92 180)
 		(effects
 			(font
@@
 		)
 	)
-	(hierarchical_label "DDR_DQS_0_P"
+	(hierarchical_label "DDR_DQS_1_P"
 		(shape bidirectional)
 		(at 101.6 109.22 180)

Commit message: power
Parts:
- R601, R602: value 100 1% -> 100
Changed lines of the file:
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@@
 			)
 		)
-		(property "Value" "100 1%"
+		(property "Value" "100"
 			(at 246.38 126.9999 0)
 			(show_name no)
@@
 			)
 		)
-		(property "Value" "100 1%"
+		(property "Value" "100"
 			(at 246.38 142.2399 0)
 			(show_name no)
