File: pcb/sch/soc-dram.kicad_sch (KiCad schematic)
At the start: 35 parts, among them U2 MT41K256M16

Commit message: byte swapping and rough layout
Other:
- moved on the sheet: C801, C802, C803, C804, C805, C806, C807, C808, R801, R802, R803, R804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

Commit message: power
Parts:
- R825: value 100 1% -> 100
- R826: value 240 1% -> 240
Changed lines of the file:
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@@
 			)
 		)
-		(property "Value" "240 1%"
+		(property "Value" "240"
 			(at 186.69 123.19 90)
 			(show_name no)
@@
 			)
 		)
-		(property "Value" "100 1%"
+		(property "Value" "100"
 			(at 93.98 127 0)
 			(show_name no)
