File: pcb/sch/soc.kicad_sch (KiCad schematic)
At the start: 2 parts

Commit message: byte swapping and rough layout
Other:
- sheet SoC 500, 501 ports: added BOOT_MODE, ETH0{RGMII}; removed ETH0{ETH}
Changed lines of the file:
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@@
+		)
+	)
+	(bus
+		(pts
+			(xy 88.9 76.2) (xy 58.42 76.2)
+		)
+		(stroke
+			(width 0)
+			(type default)
 		)
 	)
@@
 		)
 	)
+	(wire
+		(pts
+			(xy 58.42 157.48) (xy 88.9 157.48)
+		)
+		(stroke
+			(width 0)
+			(type default)
+		)
+	)
+	(wire
+		(pts
+			(xy 139.7 86.36) (xy 193.04 86.36)
+		)
+		(stroke
+			(width 0)
+			(type default)
+		)
+	)
+	(wire
+		(pts
+			(xy 139.7 50.8) (xy 193.04 50.8)
+		)
+		(stroke
+			(width 0)
+			(type default)
+		)
+	)
+	(wire
+		(pts
+			(xy 139.7 78.74) (xy 193.04 78.74)
+		)
+		(stroke
+			(width 0)
+			(type default)
+		)
+	)
+	(wire
+		(pts
+			(xy 139.7 68.58) (xy 193.04 68.58)
+		)
+		(stroke
+			(width 0)
+			(type default)
+		)
+	)
 	(bus
 		(pts
-			(xy 58.42 76.2) (xy 88.9 76.2)
-		)
-		(stroke
-			(width 0)
-			(type default)
-		)
-	)
-	(wire
-		(pts
-			(xy 58.42 157.48) (xy 88.9 157.48)
-		)
-		(stroke
-			(width 0)
-			(type default)
-		)
-	)
-	(wire
-		(pts
-			(xy 139.7 86.36) (xy 193.04 86.36)
-		)
-		(stroke
-			(width 0)
-			(type default)
-		)
-	)
-	(wire
-		(pts
-			(xy 139.7 50.8) (xy 193.04 50.8)
-		)
-		(stroke
-			(width 0)
-			(type default)
-		)
-	)
-	(wire
-		(pts
-			(xy 139.7 78.74) (xy 193.04 78.74)
-		)
-		(stroke
-			(width 0)
-			(type default)
-		)
-	)
-	(wire
-		(pts
-			(xy 139.7 68.58) (xy 193.04 68.58)
+			(xy 139.7 38.1) (xy 193.04 38.1)
 		)
 		(stroke
@@
 	(bus
 		(pts
-			(xy 139.7 38.1) (xy 193.04 38.1)
+			(xy 58.42 38.1) (xy 88.9 38.1)
+		)
+		(stroke
+			(width 0)
+			(type default)
+		)
+	)
+	(wire
+		(pts
+			(xy 139.7 81.28) (xy 193.04 81.28)
+		)
+		(stroke
+			(width 0)
+			(type default)
+		)
+	)
+	(wire
+		(pts
+			(xy 58.42 142.24) (xy 88.9 142.24)
 		)
 		(stroke
@@
 	(bus
 		(pts
-			(xy 58.42 38.1) (xy 88.9 38.1)
-		)
-		(stroke
-			(width 0)
-			(type default)
-		)
-	)
-	(wire
-		(pts
-			(xy 139.7 81.28) (xy 193.04 81.28)
-		)
-		(stroke
-			(width 0)
-			(type default)
-		)
-	)
-	(wire
-		(pts
-			(xy 58.42 142.24) (xy 88.9 142.24)
+			(xy 139.7 43.18) (xy 193.04 43.18)
+		)
+		(stroke
+			(width 0)
+			(type default)
+		)
+	)
+	(wire
+		(pts
+			(xy 228.6 119.38) (xy 238.76 119.38)
 		)
 		(stroke
@@
 	(bus
 		(pts
-			(xy 139.7 43.18) (xy 193.04 43.18)
-		)
-		(stroke
-			(width 0)
-			(type default)
-		)
-	)
-	(wire
-		(pts
-			(xy 228.6 119.38) (xy 238.76 119.38)
-		)
-		(stroke
-			(width 0)
-			(type default)
-		)
-	)
-	(bus
-		(pts
 			(xy 58.42 60.96) (xy 88.9 60.96)
+		)
+		(stroke
+			(width 0)
+			(type default)
+		)
+	)
+	(wire
+		(pts
+			(xy 58.42 91.44) (xy 88.9 91.44)
 		)
 		(stroke
@@
 		(shape bidirectional)
 		(at 58.42 60.96 180)
+		(effects
+			(font
+				(size 1.27 1.27)
+			)
+			(justify right)
+		)
+	)
+	(hierarchical_label "BOOT_MODE"
+		(shape input)
+		(at 58.42 91.44 180)
 		(effects
 			(font
@@
 			)
 		)
-		(pin "ETH0{ETH}" bidirectional
-			(at 88.9 76.2 180)
-			(effects
-				(font
-					(size 1.27 1.27)
-				)
-				(justify left)
-			)
-		)
 		(pin "1V8_FD" input
 			(at 88.9 96.52 180)
@@
 			(effects
 				(font
+					(size 1.27 1.27)
+				)
+				(justify left)
+			)
+		)
+		(pin "BOOT_MODE" input
+			(at 88.9 91.44 180)
+			(effects
+				(font
+					(size 1.27 1.27)
+				)
+				(justify left)
+			)
+		)
+		(pin "ETH0{RGMII}" bidirectional
+			(at 88.9 76.2 180)
+			(effects
+				(font

Commit message: power
Other:
- sheet FPGA 0, 13, 33 ports: added 1V8_Z, 2V5_Z, 3V3_Z; removed 1V8_FD, 2V5_FD, 3V3_FD
- sheet SoC 500, 501 ports: added 1V8_Z, 3V3_Z; removed 1V8_FD, 3V3_FD
- sheet SoC Power ports: added 1V8_Z; removed 1V8_FD
Changed lines of the file:
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@@
 		)
 	)
-	(hierarchical_label "1V8_FD"
+	(hierarchical_label "1V8_Z"
 		(shape input)
 		(at 58.42 137.16 180)
@@
 		)
 	)
-	(hierarchical_label "2V5_FD"
+	(hierarchical_label "2V5_Z"
 		(shape input)
 		(at 58.42 139.7 180)
@@
 		)
 	)
-	(hierarchical_label "1V8_FD"
+	(hierarchical_label "1V8_Z"
 		(shape input)
 		(at 58.42 162.56 180)
@@
 		)
 	)
-	(hierarchical_label "1V8_FD"
+	(hierarchical_label "1V8_Z"
 		(shape input)
 		(at 58.42 96.52 180)
@@
 		)
 	)
-	(hierarchical_label "3V3_FD"
+	(hierarchical_label "3V3_Z"
 		(shape input)
 		(at 58.42 142.24 180)
@@
 		)
 	)
-	(hierarchical_label "1V0_FD"
+	(hierarchical_label "1V0_Z"
 		(shape input)
 		(at 58.42 157.48 180)
@@
 		)
 	)
-	(hierarchical_label "3V3_FD"
+	(hierarchical_label "3V3_Z"
 		(shape input)
 		(at 58.42 99.06 180)
@@
 			)
 		)
-		(pin "1V8_FD" input
+		(pin "1V8_Z" input
 			(at 88.9 162.56 180)
 			(effects
@@
 			)
 		)
-		(pin "1V8_FD" input
+		(pin "1V8_Z" input
 			(at 88.9 137.16 180)
 			(effects
@@
 			)
 		)
-		(pin "3V3_FD" input
+		(pin "3V3_Z" input
 			(at 88.9 142.24 180)
 			(effects
@@
 			)
 		)
-		(pin "2V5_FD" input
+		(pin "2V5_Z" input
 			(at 88.9 139.7 180)
 			(effects
@@
 			)
 		)
-		(pin "3V3_FD" input
+		(pin "3V3_Z" input
 			(at 88.9 99.06 180)
 			(effects
@@
 			)
 		)
-		(pin "1V8_FD" input
+		(pin "1V8_Z" input
 			(at 88.9 96.52 180)
 			(effects
